Commit message: Gazebo sim controls
Added simple diff_drive controls to drive virtual robot in gazebo. Also added new obstacles world file. Added Rviz config file for odem frame

File: description/robot.urdf.xacro (robot description, xacro)
@@ -1,5 +1,6 @@
 <?xml version="1.0"?>
-<robot xmlns:xacro="http://www.ros.org/wiki/xacro"  name="robot">
+<robot xmlns:xacro="http://www.ros.org/wiki/xacro" name = "robot">
     <!-- Example link -->
     <xacro:include filename = "robot_core.xacro"/>
+    <xacro:include filename = "gazebo_control.xacro"/>
 </robot>

File: description/robot_core.xacro (robot description, xacro)
@@ -42,4 +42,7 @@
         </xacro:inertial_box>
     </link>
+    <gazebo reference = "chassis">
+        <material>Gazebo/FlatBlack</material>
+    </gazebo>
 <!-- LEFT WHEEL LINK -->
     <joint name="left_wheel_joint" type="continuous">
@@ -65,4 +68,7 @@
         </xacro:inertial_cylinder>
     </link>
+    <gazebo reference = "left_wheel">
+        <material>Gazebo/GreenGlow</material>
+    </gazebo>
 <!-- RIGHT WHEEL LINK -->
     <joint name="right_wheel_joint" type="continuous">
@@ -88,4 +94,7 @@
         </xacro:inertial_cylinder>
     </link>
+    <gazebo reference = 'right_wheel'>
+        <material>Gazebo/GreenGlow</material>
+    </gazebo>
 <!-- CASTOR WHEEL LINK -->
     <joint name = "castor_wheel_joint" type = "fixed">
@@ -110,3 +119,8 @@
         </xacro:inertial_sphere>
     </link>
+    <gazebo reference = "castor_wheel">
+        <material>PR2/Black</material>
+        <mu1 value = "0.001"/>
+        <mu2 value = "0.001"/>
+    </gazebo>
 </robot>
